File: I_Vilevka_MultiVib/I_Vilevka_MultiVib.sch (KiCad schematic (older format))
At the start: 11 parts

Commit message: Add files via upload
Version 2.0
Parts:
- removed Q? (x2): BC548, Package_TO_SOT_THT:TO-92_Inline, symbol Transistor_BJT:BC548
- added U1: BC847BS, symbol BC847BS:BC847BS
- gave numbers to parts that had none: 9
Connections:
- net at BT1.2 (-): now also U1.1 (E_TR2), U1.6 (E_TR1)
- net at C1.1, R1.2: now also U1.3 (C_TR1)
- net at C1.2, R2.2: now also U1.2 (B_TR2)
- net at C2.2, R3.2: now also U1.5 (B_TR1)
- net at C2.1, R4.1: now also U1.4 (C_TR2)
Changed lines of the file:
@@
 $EndDescr
 $Comp
-L Device:Battery BT?
+L Device:Battery BT1
 U 1 1 5FB2F7EE
 P 3330 3990
-F 0 "BT?" H 3438 4036 50  0000 L CNN
+F 0 "BT1" H 3438 4036 50  0000 L CNN
 F 1 "9V" H 3438 3945 50  0000 L CNN
 F 2 "" V 3330 4050 50  0001 C CNN
@@
 $EndComp
 $Comp
-L Device:LED D?
+L Device:LED D1
 U 1 1 5FB30770
 P 4000 3350
-F 0 "D?" H 4050 3460 50  0000 R CNN
+F 0 "D1" H 4050 3460 50  0000 R CNN
 F 1 "LED" H 4070 3220 50  0000 R CNN
 F 2 "" H 4000 3350 50  0001 C CNN
@@
 $EndComp
 $Comp
-L Device:R R?
+L Device:R R1
 U 1 1 5FB3126A
 P 4000 3850
-F 0 "R?" V 4090 3800 50  0000 L CNN
+F 0 "R1" V 4090 3800 50  0000 L CNN
 F 1 "470R" V 4030 3750 50  0000 L BNN
 F 2 "" V 3930 3850 50  0001 C CNN
@@
 $EndComp
 $Comp
-L Device:R R?
+L Device:R R2
 U 1 1 5FB31832
 P 4600 3850
-F 0 "R?" V 4700 3800 50  0000 L CNN
+F 0 "R2" V 4700 3800 50  0000 L CNN
 F 1 "47K" V 4600 3780 50  0000 L CNN
 F 2 "" V 4530 3850 50  0001 C CNN
@@
 $EndComp
 $Comp
-L Device:R R?
+L Device:R R3
 U 1 1 5FB34A20
 P 5100 3850
-F 0 "R?" V 5190 3800 50  0000 L CNN
+F 0 "R3" V 5190 3800 50  0000 L CNN
 F 1 "47K" V 5100 3780 50  0000 L CNN
 F 2 "" V 5030 3850 50  0001 C CNN
@@
 $EndComp
 $Comp
-L Device:R R?
+L Device:R R4
 U 1 1 5FB34A26
 P 5700 3850
-F 0 "R?" V 5600 3890 50  0000 R CNN
+F 0 "R4" V 5600 3890 50  0000 R CNN
 F 1 "470R" V 5690 3950 50  0000 R CNN
 F 2 "" V 5630 3850 50  0001 C CNN
@@
 $EndComp
 $Comp
-L Device:LED D?
+L Device:LED D2
 U 1 1 5FB35562
 P 5700 3350
-F 0 "D?" H 5760 3460 50  0000 R CNN
+F 0 "D2" H 5760 3460 50  0000 R CNN
 F 1 "LED" H 5770 3210 50  0000 R CNN
 F 2 "" H 5700 3350 50  0001 C CNN
@@
 	5100 3200 5700 3200
 $Comp
-L Device:CP1 C?
+L Device:CP1 C1
 U 1 1 5FB364DB
 P 4450 4400
-F 0 "C?" H 4520 4520 50  0000 C CNN
+F 0 "C1" H 4520 4520 50  0000 C CNN
 F 1 "47uF" H 4580 4290 50  0000 C CNN
 F 2 "" H 4450 4400 50  0001 C CNN
@@
 $EndComp
 $Comp
-L Device:CP1 C?
+L Device:CP1 C2
 U 1 1 5FB38831
 P 5250 4410
-F 0 "C?" H 5320 4510 50  0000 C CNN
+F 0 "C2" H 5320 4510 50  0000 C CNN
 F 1 "47uF" H 5370 4320 50  0000 C CNN
 F 2 "" H 5250 4410 50  0001 C CNN
@@
 	0    1    1    0
 $EndComp
-$Comp
-L Transistor_BJT:BC548 Q?
-U 1 1 5FB39521
-P 5600 4780
-F 0 "Q?" H 5791 4826 50  0000 L CNN
-F 1 "BC548" H 5791 4735 50  0000 L CNN
-F 2 "Package_TO_SOT_THT:TO-92_Inline" H 5800 4705 50  0001 L CIN
-F 3 "https://www.onsemi.com/pub/Collateral/BC550-D.pdf" H 5600 4780 50  0001 L CNN
-	1    5600 4780
-	1    0    0    -1
-$EndComp
-$Comp
-L Transistor_BJT:BC548 Q?
-U 1 1 5FB3D009
-P 4100 4790
-F 0 "Q?" H 4291 4836 50  0000 L CNN
-F 1 "BC548" H 4291 4745 50  0000 L CNN
-F 2 "Package_TO_SOT_THT:TO-92_Inline" H 4300 4715 50  0001 L CIN
-F 3 "https://www.onsemi.com/pub/Collateral/BC550-D.pdf" H 4100 4790 50  0001 L CNN
-	1    4100 4790
-	-1   0    0    -1
-$EndComp
 Wire Wire Line
 	4000 4000 4000 4400
@@
 	4300 4400 4000 4400
 Connection ~ 4000 4400
-Wire Wire Line
-	4000 4400 4000 4590
 Wire Wire Line
 	4600 4000 4600 4400
@@
 Connection ~ 5700 4410
 Wire Wire Line
-	5700 4410 5700 4580
-Wire Wire Line
-	5100 4410 4860 4410
-Wire Wire Line
-	4860 4410 4860 4790
-Wire Wire Line
-	4860 4790 4300 4790
-Connection ~ 5100 4410
-Wire Wire Line
-	5400 4780 5010 4780
-Wire Wire Line
-	5010 4780 5010 4510
-Wire Wire Line
-	5010 4510 4600 4510
-Wire Wire Line
-	4600 4400 4600 4510
-Connection ~ 4600 4400
-Wire Wire Line
-	5700 4980 5700 5000
-Wire Wire Line
-	5700 5000 4000 5000
-Wire Wire Line
-	4000 5000 4000 4990
-Wire Wire Line
-	4000 5000 3330 5000
-Wire Wire Line
-	3330 5000 3330 4190
-Connection ~ 4000 5000
-Wire Wire Line
 	3330 3790 3330 3200
 Wire Wire Line
 	3330 3200 4000 3200
 Connection ~ 4000 3200
+$Comp
+L BC847BS:BC847BS U1
+U 1 1 5FBC5062
+P 4850 4840
+F 0 "U1" H 4860 5050 50  0000 C CNN
+F 1 "BC847BS" H 4850 4570 50  0000 C CNN
+F 2 "" H 4850 5040 50  0001 C CNN
+F 3 "" H 4850 5040 50  0001 C CNN
+	1    4850 4840
+	1    0    0    -1
+$EndComp
+Wire Wire Line
+	5250 4940 5310 4940
+Wire Wire Line
+	5310 4940 5310 5050
+Wire Wire Line
+	5310 5050 3330 5050
+Wire Wire Line
+	3330 4190 3330 4740
+Wire Wire Line
+	4450 4740 3330 4740
+Connection ~ 3330 4740
+Wire Wire Line
+	3330 4740 3330 5050
+Wire Wire Line
+	4450 4840 4360 4840
+Wire Wire Line
+	4360 4840 4360 4560
+Wire Wire Line
+	4360 4560 4600 4560
+Wire Wire Line
+	4600 4560 4600 4400
+Connection ~ 4600 4400
+Wire Wire Line
+	5250 4840 5380 4840
+Wire Wire Line
+	5380 4840 5380 4580
+Wire Wire Line
+	5380 4580 5100 4580
+Wire Wire Line
+	5100 4580 5100 4410
+Connection ~ 5100 4410
+Wire Wire Line
+	5250 4740 5700 4740
+Wire Wire Line
+	4450 4940 4000 4940
+Wire Wire Line
+	5700 4410 5700 4740
+Wire Wire Line
+	4000 4400 4000 4940
 $EndSCHEMATC
